File: Buffered mult rev 2.sch (EAGLE design)
At the start: 31 parts, among them J1 EUROPWR_2X05-SMD, U1 TL072_SMD, U2 TL072_SMD, U3 TL072_SMD

Commit message: minor changes
Parts:
- removed OUT1, OUT2, OUT3, OUT4, OUT5, U$OUT6: THONKICONNOLD, MusicThingModular:THONKICONNOLD
- added IC1: OPA4171, linear:TL074PW
Connections:
- removed net N$16: C4.2, C6.2
- removed net N$18: C5.2, C7.2
- net GND: now also C2.1, C3.1, C4.1, C5.1, C6.1, C7.1, U1P.V+, U1P.V-, U2P.V+, U2P.V-, U3P.V+, U3P.V-; no longer C2.2, C3.2, OUT1.SLEEVE, OUT2.SLEEVE, OUT3.SLEEVE, OUT4.SLEEVE, OUT5.SLEEVE, U$OUT6.SLEEVE
- net N$1: no longer U$OUT6.TIP
- net N$10: now also IC1C.+IN, IC1C.OUT; no longer U1B.-IN, U1B.OUT
- net N$11: now also IC1B.+IN; no longer U2B.+IN, U3A.+IN, U3B.+IN
- net N$12: no longer U3B.-IN, U3B.OUT
- net N$13: no longer U3A.-IN, U3A.OUT
- net N$17: now also IC1B.-IN, IC1B.OUT; no longer U2B.-IN, U2B.OUT
- net N$2: now also IC1A.+IN, IC1A.OUT; no longer U1A.-IN, U1A.OUT
- net N$3: no longer OUT5.TIP
- net N$4: no longer OUT4.TIP
- net N$5: now also IC1A.-IN, IC1C.-IN, IC1D.-IN; no longer U1A.+IN, U1B.+IN, U2A.+IN
- net N$6: now also IC1D.+IN, IC1D.OUT; no longer U2A.-IN, U2A.OUT
- net N$7: no longer OUT2.TIP
- net N$8: no longer OUT3.TIP
- net N$9: no longer OUT1.TIP
- net VCC: no longer C2.1, C4.1, C5.1, U1P.V+, U2P.V+, U3P.V+
- net VEE: no longer C3.1, C6.1, C7.1, U1P.V-, U2P.V-, U3P.V-
