File: Buffered mult rev 3.sch (EAGLE design)
At the start: 28 parts, among them IC1 OPA4171, IC2 OPA2171, J1 EURO_POWER_HEADERFAT_PADS

Commit message: Finalized design, generated Gerbers.
Parts:
- removed IC2: OPA2171, linear:TL072D
- removed IN2, OUT4: PJ302M, pj302m:PJ302M
- added IC3: OPA4171, linear:TL074PW
- added IN2/OUT4, OUT7: PJ302M, pj302m:PJ302M
- added R9: 1k, SparkFun-Passives:RESISTOR1206
Connections:
- removed net N$11: IC1B.+IN, IC2A.-IN, IC2B.+IN, R8.2
- new net N$16: IC1D.-IN, IC1D.OUT, R9.1
- new net N$18: IN2/OUT4.SWITCH, R9.2
- new net N$19: IC3A.+IN, IC3B.+IN, IC3C.+IN, IN2/OUT4.TIP, R8.2
- net GND: now also IC3D.+IN, IC3D.-IN, IC3D.OUT, IN2/OUT4.SLEEVE, OUT7.SLEEVE; no longer IN2.SLEEVE, OUT4.SLEEVE
- net N$1: now also OUT7.TIP; no longer OUT6.TIP
- net N$10: now also IC1B.-IN, IC1B.OUT; no longer IC1C.+IN, IC1C.OUT
- net N$12: now also IC3C.-IN, IC3C.OUT; no longer IC2A.OUT
- net N$13: now also IC3B.-IN, IC3B.OUT; no longer IC2B.-IN, IC2B.OUT
- net N$17: now also IC3A.-IN, IC3A.OUT; no longer IC1B.-IN, IC1B.OUT
- net N$3: now also OUT6.TIP; no longer OUT5.TIP
- net N$4: now also OUT5.TIP; no longer OUT4.TIP
- net N$5: now also IC1B.+IN, IC1C.+IN, IC1D.+IN; no longer IC1C.-IN, IC1D.-IN, IN2.SWITCH, IN2.TIP
- net N$6: now also IC1C.-IN, IC1C.OUT; no longer IC1D.+IN, IC1D.OUT
- net VCC: now also IC3P.V+; no longer IC2P.V+
- net VEE: now also IC3P.V-; no longer IC2P.V-
Other:
- note added: "If jack is inserted, this and the following jacks serve as a 1:3 mult, otherwise they are 4 outputs part of the total 1:7 mult"
- moved on the sheet: IC1B, IC1C, IC1D, OUT5, OUT6
